Commit message: edited  golf_club urdf

File: src/apex_putter/urdf/golf_club/urdf/golf_club.urdf (robot description, URDF)
Before this commit: robot golb_club_fixed, 1 links, 0 joints
Links:
- link base_link: geometry collision mesh filename=package://golf_club/meshes/base_link.STL; visual mesh filename=package://golf_club/meshes/base_link.STL
